File: frontendboard.sch (EAGLE design)
At the start: 64 parts, among them U1 MAX2769, X3 BU-SMA-H

Commit message: All ERC errors and warnings fixed or approved. No LEDs in place.
Parts:
- C10, C11: value (none) -> 10nF
Connections:
- net BAR_GND: now also Q2.2; no longer Q2.1
- net N$3: now also Q2.1; no longer Q2.2
Other:
- moved on the sheet: C11, Q2
Changed lines of the file:
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@@
 <part name="DIG_GND5" library="supply" deviceset="GND_BAR" device="" value="GND"/>
 <part name="C9" library="rcl_custom" deviceset="C-EU" device="0603-B" value="0.1uF"/>
-<part name="C10" library="rcl_custom" deviceset="C-EU" device="0603-B"/>
-<part name="C11" library="rcl_custom" deviceset="C-EU" device="0603-B"/>
+<part name="C10" library="rcl_custom" deviceset="C-EU" device="0603-B" value="10nF"/>
+<part name="C11" library="rcl_custom" deviceset="C-EU" device="0603-B" value="10nF"/>
 <part name="DIG_GND8" library="supply" deviceset="GND_BAR" device="" value="GND"/>
 <part name="DIG_GND9" library="supply" deviceset="GND_BAR" device="" value="GND"/>
@@
 <part name="DIG_GND25" library="supply" deviceset="GND_BAR" device="" value="GND"/>
 <part name="R7" library="rcl_custom" deviceset="R-US_" device="0603-B" value="1.5k"/>
-<part name="3.3VD" library="SparkFun" deviceset="3.3V" device="" value="3.3VD"/>
-<part name="3.3VD2" library="SparkFun" deviceset="3.3V" device="" value="3.3VD"/>
 <part name="DIG_GND10" library="supply" deviceset="GND_BAR" device="" value="GND"/>
 <part name="DIG_GND26" library="supply" deviceset="GND_BAR" device="" value="GND"/>
@@
 <part name="C1" library="rcl_custom" deviceset="C-EU" device="0603-B" value="2.2uF"/>
 <part name="DIG_GND17" library="supply" deviceset="GND_BAR" device="" value="GND"/>
-<part name="3.3VD5" library="SparkFun" deviceset="3.3V" device="" value="3.3VD"/>
 <part name="R1" library="rcl_custom" deviceset="R-US_" device="0603-B" value="1k"/>
 <part name="R8" library="rcl_custom" deviceset="R-US_" device="0603-B" value="1k"/>
-<part name="3.3VD6" library="SparkFun" deviceset="3.3V" device="" value="3.3VD"/>
 <part name="DIG_GND30" library="supply" deviceset="GND_BAR" device="" value="GND"/>
 <part name="C23" library="rcl_custom" deviceset="C-EU" device="0603-B" value="2.2uF"/>
@@
 <part name="C39" library="rcl_custom" deviceset="C-EU" device="0603-B" value="1uF"/>
 <part name="DIG_GND53" library="supply" deviceset="GND_BAR" device="" value="GND"/>
-<part name="Q2" library="crystal" deviceset="CRYSTAL" device="CTS406"/>
-<part name="DIG_GND7" library="supply" deviceset="GND_BAR" device="" value="GND"/>
 <part name="C20" library="rcl_custom" deviceset="C-EU" device="0603-B" value="2.2uF"/>
 <part name="DIG_GND20" library="supply" deviceset="GND_BAR" device="" value="GND"/>
@@
 <part name="U$28" library="SparkFun-Aesthetics" deviceset="3.3VA" device=""/>
 <part name="DIG_GND22" library="supply" deviceset="GND_BAR" device="" value="GND"/>
+<part name="Q2" library="crystal" deviceset="CRYSTAL" device="CTS406"/>
+<part name="DIG_GND7" library="supply" deviceset="GND_BAR" device="" value="GND"/>
+<part name="U$29" library="SparkFun-Aesthetics" deviceset="3.3VD" device=""/>
+<part name="U$30" library="SparkFun-Aesthetics" deviceset="3.3VD" device=""/>
+<part name="U$31" library="SparkFun-Aesthetics" deviceset="3.3VD" device=""/>
+<part name="U$32" library="SparkFun-Aesthetics" deviceset="3.3VD" device=""/>
 </parts>
 <sheets>
@@
 <instance part="C9" gate="CE" x="675.64" y="157.48" rot="MR0"/>
 <instance part="C10" gate="CE" x="701.04" y="160.02"/>
-<instance part="C11" gate="CE" x="706.12" y="137.16"/>
+<instance part="C11" gate="CE" x="718.82" y="172.72"/>
 <instance part="DIG_GND8" gate="1" x="701.04" y="152.4"/>
 <instance part="DIG_GND9" gate="1" x="675.64" y="149.86" rot="MR0"/>
@@
 <instance part="DIG_GND25" gate="1" x="25.4" y="50.8" rot="MR0"/>
 <instance part="R7" gate="R" x="45.72" y="81.28" rot="MR90"/>
-<instance part="3.3VD" gate="G$1" x="45.72" y="99.06" rot="MR0"/>
-<instance part="3.3VD2" gate="G$1" x="675.64" y="162.56" rot="MR0"/>
 <instance part="DIG_GND10" gate="1" x="218.44" y="121.92"/>
 <instance part="DIG_GND26" gate="1" x="223.52" y="88.9"/>
@@
 <instance part="C1" gate="CE" x="170.18" y="99.06" rot="R180"/>
 <instance part="DIG_GND17" gate="1" x="170.18" y="93.98"/>
-<instance part="3.3VD5" gate="G$1" x="93.98" y="99.06"/>
 <instance part="R1" gate="R" x="76.2" y="88.9" rot="R90"/>
 <instance part="R8" gate="R" x="76.2" y="76.2" rot="R90"/>
-<instance part="3.3VD6" gate="G$1" x="76.2" y="99.06"/>
 <instance part="DIG_GND30" gate="1" x="76.2" y="68.58"/>
 <instance part="C23" gate="CE" x="63.5" y="73.66" rot="R180"/>
@@
 <instance part="C39" gate="CE" x="215.9" y="68.58" rot="R180"/>
 <instance part="DIG_GND53" gate="1" x="215.9" y="58.42"/>
-<instance part="Q2" gate="G$1" x="741.68" y="165.1"/>
-<instance part="DIG_GND7" gate="1" x="731.52" y="162.56"/>
 <instance part="C20" gate="CE" x="154.94" y="134.62" rot="R180"/>
 <instance part="DIG_GND20" gate="1" x="154.94" y="129.54"/>
@@
 <instance part="U$28" gate="3.3VA" x="568.96" y="96.52"/>
 <instance part="DIG_GND22" gate="1" x="721.36" y="81.28"/>
+<instance part="Q2" gate="G$1" x="718.82" y="160.02" rot="R270"/>
+<instance part="DIG_GND7" gate="1" x="718.82" y="149.86"/>
+<instance part="U$29" gate="3.3VD" x="45.72" y="99.06"/>
+<instance part="U$30" gate="3.3VD" x="76.2" y="99.06"/>
+<instance part="U$31" gate="3.3VD" x="93.98" y="99.06"/>
+<instance part="U$32" gate="3.3VD" x="675.64" y="162.56"/>
 </instances>
 <busses>
@@
 </segment>
 <segment>
-<wire x1="739.14" y1="165.1" x2="731.52" y2="165.1" width="0.1524" layer="91"/>
-<pinref part="Q2" gate="G$1" pin="1"/>
-<pinref part="DIG_GND7" gate="1" pin="BAR_GND"/>
-</segment>
-<segment>
 <pinref part="C20" gate="CE" pin="1"/>
 <pinref part="DIG_GND20" gate="1" pin="BAR_GND"/>
@@
 <wire x1="721.36" y1="86.36" x2="721.36" y2="83.82" width="0.1524" layer="91"/>
 <pinref part="DIG_GND22" gate="1" pin="BAR_GND"/>
+</segment>
+<segment>
+<pinref part="Q2" gate="G$1" pin="2"/>
+<wire x1="718.82" y1="157.48" x2="718.82" y2="152.4" width="0.1524" layer="91"/>
+<pinref part="DIG_GND7" gate="1" pin="BAR_GND"/>
 </segment>
 </net>
@@
 <segment>
 <wire x1="701.04" y1="129.54" x2="701.04" y2="139.7" width="0.1524" layer="91"/>
-<wire x1="701.04" y1="139.7" x2="706.12" y2="139.7" width="0.1524" layer="91"/>
+<wire x1="701.04" y1="139.7" x2="711.2" y2="139.7" width="0.1524" layer="91"/>
+<wire x1="711.2" y1="139.7" x2="711.2" y2="175.26" width="0.1524" layer="91"/>
+<wire x1="711.2" y1="175.26" x2="718.82" y2="175.26" width="0.1524" layer="91"/>
 <pinref part="U1" gate="G$1" pin="XTAL"/>
 <pinref part="C11" gate="CE" pin="1"/>
@@
 <pinref part="C9" gate="CE" pin="1"/>
 <pinref part="U1" gate="G$1" pin="VCCADC"/>
-<pinref part="3.3VD2" gate="G$1" pin="3.3V"/>
+<pinref part="U$32" gate="3.3VD" pin="3.3VD"/>
 </segment>
 <segment>
@@
 <segment>
 <pinref part="R7" gate="R" pin="2"/>
-<pinref part="3.3VD" gate="G$1" pin="3.3V"/>
 <wire x1="45.72" y1="99.06" x2="45.72" y2="86.36" width="0.1524" layer="91"/>
+<pinref part="U$29" gate="3.3VD" pin="3.3VD"/>
 </segment>
 <segment>
 <wire x1="76.2" y1="93.98" x2="76.2" y2="99.06" width="0.1524" layer="91"/>
 <pinref part="R1" gate="R" pin="2"/>
-<pinref part="3.3VD6" gate="G$1" pin="3.3V"/>
+<pinref part="U$30" gate="3.3VD" pin="3.3VD"/>
 </segment>
 <segment>
@@
 <junction x="93.98" y="86.36"/>
 <pinref part="C28" gate="CE" pin="2"/>
-<pinref part="3.3VD5" gate="G$1" pin="3.3V"/>
 <pinref part="HS_USB" gate="G$1" pin="VDDIO"/>
+<pinref part="U$31" gate="3.3VD" pin="3.3VD"/>
 </segment>
 <segment>
@@
 <net name="N$3" class="0">
 <segment>
-<wire x1="706.12" y1="132.08" x2="706.12" y2="129.54" width="0.1524" layer="91"/>
-<wire x1="706.12" y1="129.54" x2="716.28" y2="129.54" width="0.1524" layer="91"/>
-<wire x1="716.28" y1="129.54" x2="716.28" y2="142.24" width="0.1524" layer="91"/>
-<wire x1="716.28" y1="142.24" x2="749.3" y2="142.24" width="0.1524" layer="91"/>
-<wire x1="749.3" y1="142.24" x2="749.3" y2="165.1" width="0.1524" layer="91"/>
-<wire x1="749.3" y1="165.1" x2="744.22" y2="165.1" width="0.1524" layer="91"/>
+<wire x1="718.82" y1="167.64" x2="718.82" y2="162.56" width="0.1524" layer="91"/>
 <pinref part="C11" gate="CE" pin="2"/>
-<pinref part="Q2" gate="G$1" pin="2"/>
+<pinref part="Q2" gate="G$1" pin="1"/>
 </segment>
 </net>
@@
 </sheet>
 </sheets>
+<errors>
+</errors>
 </schematic>
 </drawing>

Commit message: Start layout on RF side.
Parts:
- C10, C11, C12, C13, C14, C15, C16, C17, C18, C19, C22, C24, C25, C3, C4, C5, C6, C7, C8, C9: device rcl_custom:C-EU0603-B -> rcl:C-EUC0402
- R2, R3, R4, R5, R6: device rcl_custom:R-US_0603-B -> rcl:R-US_R0402
